Commit message: 250702

File: realman_cable/urdf/rm_75b_hand_gripper.urdf (robot description, URDF)
Before this commit: robot rm_75_6f_description, 11 links, 10 joints
Links:
- removed link robotiq
- added link left_robotiq
- added link right_robotiq
Joints:
- removed joint joint_robotiq
- added joint left_joint_robotiq: type fixed, parent Link7, child left_robotiq, origin xyz=0 0 0.19182 rpy=0 0 2.8780
- added joint right_joint_robotiq: type fixed, parent Link7, child right_robotiq, origin xyz=0 0 0.22032 rpy=0 -2.356 1.047
